File: pmod-composite/pmod-composite.kicad_pcb (KiCad board)
At the start: 2 copper layers, 37.1 x 66.5 mm, 36 parts, among them J1 Conn_02x06_Top_Bottom, J2 PJRAN1X1U04X, J3 PJRAN1X1U04X, U1 NE5532

Commit message: route board
Parts:
- J1: footprint Connector_PinHeader_1.00mm:PinHeader_2x06_P1.00mm_Vertical -> Connector_PinHeader_2.54mm:PinHeader_2x06_P2.54mm_Vertical
- moved R1 13.1 mm to (53.8, 37.6), turned to 180 degrees
- moved R4 13.1 mm to (53.8, 48.3), turned to 180 degrees
- moved R2 8.44 mm to (53.9, 41.1), turned to 180 degrees
- moved R3 8.44 mm to (53.9, 44.7), turned to 180 degrees
- moved C4 4.85 mm to (44.2, 75.7)
- moved J1 3.85 mm to (50.8, 31.5)
Routing:
- net +3V3: track 0.00 -> 73.8 mm
- net Net-(C1-Pad1): track 0.00 -> 46.0 mm
- net Net-(C2-Pad1): track 0.00 -> 41.7 mm
- net Net-(C8-Pad1): track 0.00 -> 25.6 mm
- net Net-(C7-Pad1): track 0.00 -> 25.2 mm
- net P1_4: track 0.00 -> 22.2 mm
- net Net-(C4-Pad1): track 0.00 -> 18.9 mm
- net P1_3: track 0.00 -> 17.6 mm
- net P1_10: track 0.00 -> 15.5 mm
- net Net-(C3-Pad1): track 0.00 -> 13.3 mm
- net P1_2: track 0.00 -> 13.0 mm
- net Net-(R14-Pad1): track 0.00 -> 13.0 mm
- net P1_9: track 0.00 -> 12.0 mm
- net P1_7: track 0.00 -> 11.9 mm
- net Net-(C12-Pad2): track 0.00 -> 11.9 mm
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Other:
- board size 37.1 x 66.5 mm -> 37.1 x 67.1 mm
